Commit message: separated 120id and 120id12l (120id12l needs updated meshes and joint poses)

File: fanuc_arcmate120id_support/urdf/arcmate120id_macro.xacro (robot description, xacro)
@@ -2,5 +2,5 @@
 <robot xmlns:xacro="http://wiki.ros.org/xacro">
   <xacro:include filename="$(find fanuc_resources)/urdf/common_materials.xacro"/>
-  <xacro:macro name="fanuc_arcmate120id12" params="prefix">
+  <xacro:macro name="fanuc_arcmate120id" params="prefix">
     <!-- links: main serial chain -->
     <link name="${prefix}base_link">
@@ -8,5 +8,5 @@
         <origin xyz="0 0 0" rpy="0 0 0"/>
         <geometry>
-          <mesh filename="package://fanuc_arcmate120id12_support/meshes/arcmate120id12/visual/base_link.stl"/>
+          <mesh filename="package://fanuc_arcmate120id_support/meshes/arcmate120id/visual/base_link.stl"/>
         </geometry>
         <xacro:material_fanuc_black/>
@@ -15,5 +15,5 @@
         <origin xyz="0 0 0" rpy="0 0 0"/>
         <geometry>
-          <mesh filename="package://fanuc_arcmate120id12_support/meshes/arcmate120id12/collision/base_link.stl"/>
+          <mesh filename="package://fanuc_arcmate120id_support/meshes/arcmate120id/collision/base_link.stl"/>
         </geometry>
       </collision>
@@ -23,5 +23,5 @@
         <origin xyz="0 0 0" rpy="0 0 0"/>
         <geometry>
-          <mesh filename="package://fanuc_arcmate120id12_support/meshes/arcmate120id12/visual/link_1.stl"/>
+          <mesh filename="package://fanuc_arcmate120id_support/meshes/arcmate120id/visual/link_1.stl"/>
         </geometry>
         <xacro:material_fanuc_yellow/>
@@ -30,5 +30,5 @@
         <origin xyz="0 0 0" rpy="0 0 0"/>
         <geometry>
-          <mesh filename="package://fanuc_arcmate120id12_support/meshes/arcmate120id12/collision/link_1.stl"/>
+          <mesh filename="package://fanuc_arcmate120id_support/meshes/arcmate120id/collision/link_1.stl"/>
         </geometry>
       </collision>
@@ -38,5 +38,5 @@
         <origin xyz="0 0 0" rpy="0 0 0"/>
         <geometry>
-          <mesh filename="package://fanuc_arcmate120id12_support/meshes/arcmate120id12/visual/link_2.stl"/>
+          <mesh filename="package://fanuc_arcmate120id_support/meshes/arcmate120id/visual/link_2.stl"/>
         </geometry>
         <xacro:material_fanuc_black/>
@@ -45,5 +45,5 @@
         <origin xyz="0 0 0" rpy="0 0 0"/>
         <geometry>
-          <mesh filename="package://fanuc_arcmate120id12_support/meshes/arcmate120id12/collision/link_2.stl"/>
+          <mesh filename="package://fanuc_arcmate120id_support/meshes/arcmate120id/collision/link_2.stl"/>
         </geometry>
       </collision>
@@ -53,5 +53,5 @@
         <origin xyz="0 0 0" rpy="0 0 0"/>
         <geometry>
-          <mesh filename="package://fanuc_arcmate120id12_support/meshes/arcmate120id12/visual/link_3.stl"/>
+          <mesh filename="package://fanuc_arcmate120id_support/meshes/arcmate120id/visual/link_3.stl"/>
         </geometry>
         <xacro:material_fanuc_yellow/>
@@ -60,5 +60,5 @@
         <origin xyz="0 0 0" rpy="0 0 0"/>
         <geometry>
-          <mesh filename="package://fanuc_arcmate120id12_support/meshes/arcmate120id12/collision/link_3.stl"/>
+          <mesh filename="package://fanuc_arcmate120id_support/meshes/arcmate120id/collision/link_3.stl"/>
         </geometry>
       </collision>
@@ -68,5 +68,5 @@
         <origin xyz="0 0 0" rpy="0 0 0"/>
         <geometry>
-          <mesh filename="package://fanuc_arcmate120id12_support/meshes/arcmate120id12/visual/link_4.stl"/>
+          <mesh filename="package://fanuc_arcmate120id_support/meshes/arcmate120id/visual/link_4.stl"/>
         </geometry>
         <xacro:material_fanuc_black/>
@@ -75,5 +75,5 @@
         <origin xyz="0 0 0" rpy="0 0 0"/>
         <geometry>
-          <mesh filename="package://fanuc_arcmate120id12_support/meshes/arcmate120id12/collision/link_4.stl"/>
+          <mesh filename="package://fanuc_arcmate120id_support/meshes/arcmate120id/collision/link_4.stl"/>
         </geometry>
       </collision>
@@ -83,5 +83,5 @@
         <origin xyz="0 0 0" rpy="0 0 0"/>
         <geometry>
-          <mesh filename="package://fanuc_arcmate120id12_support/meshes/arcmate120id12/visual/link_5.stl"/>
+          <mesh filename="package://fanuc_arcmate120id_support/meshes/arcmate120id/visual/link_5.stl"/>
         </geometry>
         <xacro:material_fanuc_yellow/>
@@ -90,5 +90,5 @@
         <origin xyz="0 0 0" rpy="0 0 0"/>
         <geometry>
-          <mesh filename="package://fanuc_arcmate120id12_support/meshes/arcmate120id12/collision/link_5.stl"/>
+          <mesh filename="package://fanuc_arcmate120id_support/meshes/arcmate120id/collision/link_5.stl"/>
         </geometry>
       </collision>
@@ -98,5 +98,5 @@
         <origin xyz="0 0 0" rpy="0 0 0"/>
         <geometry>
-          <mesh filename="package://fanuc_arcmate120id12_support/meshes/arcmate120id12/visual/link_6.stl"/>
+          <mesh filename="package://fanuc_arcmate120id_support/meshes/arcmate120id/visual/link_6.stl"/>
         </geometry>
         <xacro:material_fanuc_black/>
@@ -105,5 +105,5 @@
         <origin xyz="0 0 0" rpy="0 0 0"/>
         <geometry>
-          <mesh filename="package://fanuc_arcmate120id12_support/meshes/arcmate120id12/collision/link_6.stl"/>
+          <mesh filename="package://fanuc_arcmate120id_support/meshes/arcmate120id/collision/link_6.stl"/>
         </geometry>
       </collision>
@@ -115,5 +115,5 @@
       <child link="${prefix}link_1"/>
       <axis xyz="0 0 1"/>
-      <limit effort="0" lower="-1" upper="1" velocity="0.1"/>
+      <limit effort="0" lower="${radians(-170)}" upper="${radians(170)}" velocity="${radians(210)}"/>
     </joint>
     <joint name="${prefix}joint_2" type="revolute">
@@ -122,5 +122,5 @@
       <child link="${prefix}link_2"/>
       <axis xyz="0 0 1"/>
-      <limit effort="0" lower="-1" upper="1" velocity="0.1"/>
+      <limit effort="0" lower="${radians(-100)}" upper="${radians(160)}" velocity="${radians(210)}"/>
     </joint>
     <joint name="${prefix}joint_3" type="revolute">
@@ -129,5 +129,5 @@
       <child link="${prefix}link_3"/>
       <axis xyz="0 0 1"/>
-      <limit effort="0" lower="-1" upper="1" velocity="0.1"/>
+      <limit effort="0" lower="${radians(-190)}" upper="${radians(268.4)}" velocity="${radians(265)}"/>
     </joint>
     <joint name="${prefix}joint_4" type="revolute">
@@ -136,5 +136,5 @@
       <child link="${prefix}link_4"/>
       <axis xyz="0 0 1"/>
-      <limit effort="0" lower="-1" upper="1" velocity="0.1"/>
+      <limit effort="0" lower="${radians(-200)}" upper="${radians(200)}" velocity="${radians(420)}"/>
     </joint>
     <joint name="${prefix}joint_5" type="revolute">
@@ -143,5 +143,5 @@
       <child link="${prefix}link_5"/>
       <axis xyz="0 0 1"/>
-      <limit effort="0" lower="-1" upper="1" velocity="0.1"/>
+      <limit effort="0" lower="${radians(-140)}" upper="${radians(140)}" velocity="${radians(420)}"/>
     </joint>
     <joint name="${prefix}joint_6" type="revolute">
@@ -150,5 +150,5 @@
       <child link="${prefix}link_6"/>
       <axis xyz="0 0 1"/>
-      <limit effort="0" lower="-1" upper="1" velocity="0.1"/>
+      <limit effort="0" lower="${radians(-270)}" upper="${radians(270)}" velocity="${radians(720)}"/>
     </joint>
     <!-- ROS base_link to Fanuc World Coordinates transform -->
