Commit message: changed arcmate120id to m20id

File: fanuc_m20id_support/urdf/m20id12l_macro.xacro (robot description, xacro)
@@ -1,6 +1,8 @@
 <?xml version="1.0"?>
+<!-- ATTENTION: mesh files and joint poses currently represent the 120iD and NOT the 120iD12L -->
+<!-- TODO: update mesh files and joint poses for 120iD12L -->
 <robot xmlns:xacro="http://wiki.ros.org/xacro">
   <xacro:include filename="$(find fanuc_resources)/urdf/common_materials.xacro"/>
-  <xacro:macro name="fanuc_arcmate120id" params="prefix">
+  <xacro:macro name="fanuc_m20id12l" params="prefix">
     <!-- links: main serial chain -->
     <link name="${prefix}base_link">
@@ -8,5 +10,5 @@
         <origin xyz="0 0 0" rpy="0 0 0"/>
         <geometry>
-          <mesh filename="package://fanuc_arcmate120id_support/meshes/arcmate120id/visual/base_link.stl"/>
+          <mesh filename="package://fanuc_m20id_support/meshes/m20id12l/visual/base_link.stl"/>
         </geometry>
         <xacro:material_fanuc_black/>
@@ -15,5 +17,5 @@
         <origin xyz="0 0 0" rpy="0 0 0"/>
         <geometry>
-          <mesh filename="package://fanuc_arcmate120id_support/meshes/arcmate120id/collision/base_link.stl"/>
+          <mesh filename="package://fanuc_m20id_support/meshes/m20id12l/collision/base_link.stl"/>
         </geometry>
       </collision>
@@ -23,5 +25,5 @@
         <origin xyz="0 0 0" rpy="0 0 0"/>
         <geometry>
-          <mesh filename="package://fanuc_arcmate120id_support/meshes/arcmate120id/visual/link_1.stl"/>
+          <mesh filename="package://fanuc_m20id_support/meshes/m20id12l/visual/link_1.stl"/>
         </geometry>
         <xacro:material_fanuc_yellow/>
@@ -30,5 +32,5 @@
         <origin xyz="0 0 0" rpy="0 0 0"/>
         <geometry>
-          <mesh filename="package://fanuc_arcmate120id_support/meshes/arcmate120id/collision/link_1.stl"/>
+          <mesh filename="package://fanuc_m20id_support/meshes/m20id12l/collision/link_1.stl"/>
         </geometry>
       </collision>
@@ -38,5 +40,5 @@
         <origin xyz="0 0 0" rpy="0 0 0"/>
         <geometry>
-          <mesh filename="package://fanuc_arcmate120id_support/meshes/arcmate120id/visual/link_2.stl"/>
+          <mesh filename="package://fanuc_m20id_support/meshes/m20id12l/visual/link_2.stl"/>
         </geometry>
         <xacro:material_fanuc_black/>
@@ -45,5 +47,5 @@
         <origin xyz="0 0 0" rpy="0 0 0"/>
         <geometry>
-          <mesh filename="package://fanuc_arcmate120id_support/meshes/arcmate120id/collision/link_2.stl"/>
+          <mesh filename="package://fanuc_m20id_support/meshes/m20id12l/collision/link_2.stl"/>
         </geometry>
       </collision>
@@ -53,5 +55,5 @@
         <origin xyz="0 0 0" rpy="0 0 0"/>
         <geometry>
-          <mesh filename="package://fanuc_arcmate120id_support/meshes/arcmate120id/visual/link_3.stl"/>
+          <mesh filename="package://fanuc_m20id_support/meshes/m20id12l/visual/link_3.stl"/>
         </geometry>
         <xacro:material_fanuc_yellow/>
@@ -60,5 +62,5 @@
         <origin xyz="0 0 0" rpy="0 0 0"/>
         <geometry>
-          <mesh filename="package://fanuc_arcmate120id_support/meshes/arcmate120id/collision/link_3.stl"/>
+          <mesh filename="package://fanuc_m20id_support/meshes/m20id12l/collision/link_3.stl"/>
         </geometry>
       </collision>
@@ -68,5 +70,5 @@
         <origin xyz="0 0 0" rpy="0 0 0"/>
         <geometry>
-          <mesh filename="package://fanuc_arcmate120id_support/meshes/arcmate120id/visual/link_4.stl"/>
+          <mesh filename="package://fanuc_m20id_support/meshes/m20id12l/visual/link_4.stl"/>
         </geometry>
         <xacro:material_fanuc_black/>
@@ -75,5 +77,5 @@
         <origin xyz="0 0 0" rpy="0 0 0"/>
         <geometry>
-          <mesh filename="package://fanuc_arcmate120id_support/meshes/arcmate120id/collision/link_4.stl"/>
+          <mesh filename="package://fanuc_m20id_support/meshes/m20id12l/collision/link_4.stl"/>
         </geometry>
       </collision>
@@ -83,5 +85,5 @@
         <origin xyz="0 0 0" rpy="0 0 0"/>
         <geometry>
-          <mesh filename="package://fanuc_arcmate120id_support/meshes/arcmate120id/visual/link_5.stl"/>
+          <mesh filename="package://fanuc_m20id_support/meshes/m20id12l/visual/link_5.stl"/>
         </geometry>
         <xacro:material_fanuc_yellow/>
@@ -90,5 +92,5 @@
         <origin xyz="0 0 0" rpy="0 0 0"/>
         <geometry>
-          <mesh filename="package://fanuc_arcmate120id_support/meshes/arcmate120id/collision/link_5.stl"/>
+          <mesh filename="package://fanuc_m20id_support/meshes/m20id12l/collision/link_5.stl"/>
         </geometry>
       </collision>
@@ -98,5 +100,5 @@
         <origin xyz="0 0 0" rpy="0 0 0"/>
         <geometry>
-          <mesh filename="package://fanuc_arcmate120id_support/meshes/arcmate120id/visual/link_6.stl"/>
+          <mesh filename="package://fanuc_m20id_support/meshes/m20id12l/visual/link_6.stl"/>
         </geometry>
         <xacro:material_fanuc_black/>
@@ -105,5 +107,5 @@
         <origin xyz="0 0 0" rpy="0 0 0"/>
         <geometry>
-          <mesh filename="package://fanuc_arcmate120id_support/meshes/arcmate120id/collision/link_6.stl"/>
+          <mesh filename="package://fanuc_m20id_support/meshes/m20id12l/collision/link_6.stl"/>
         </geometry>
       </collision>
@@ -143,5 +145,5 @@
       <child link="${prefix}link_5"/>
       <axis xyz="0 0 1"/>
-      <limit effort="0" lower="${radians(-140)}" upper="${radians(140)}" velocity="${radians(420)}"/>
+      <limit effort="0" lower="${radians(-140)}" upper="${radians(140)}" velocity="${radians(450)}"/>
     </joint>
     <joint name="${prefix}joint_6" type="revolute">

File: fanuc_m20id_support/urdf/m20id_macro.xacro (robot description, xacro)
@@ -1,8 +1,6 @@
 <?xml version="1.0"?>
-<!-- ATTENTION: mesh files and joint poses currently represent the 120iD and NOT the 120iD12L -->
-<!-- TODO: update mesh files and joint poses for 120iD12L -->
 <robot xmlns:xacro="http://wiki.ros.org/xacro">
   <xacro:include filename="$(find fanuc_resources)/urdf/common_materials.xacro"/>
-  <xacro:macro name="fanuc_arcmate120id12l" params="prefix">
+  <xacro:macro name="fanuc_m20id" params="prefix">
     <!-- links: main serial chain -->
     <link name="${prefix}base_link">
@@ -10,5 +8,5 @@
         <origin xyz="0 0 0" rpy="0 0 0"/>
         <geometry>
-          <mesh filename="package://fanuc_arcmate120id_support/meshes/arcmate120id12l/visual/base_link.stl"/>
+          <mesh filename="package://fanuc_m20id_support/meshes/m20id/visual/base_link.stl"/>
         </geometry>
         <xacro:material_fanuc_black/>
@@ -17,5 +15,5 @@
         <origin xyz="0 0 0" rpy="0 0 0"/>
         <geometry>
-          <mesh filename="package://fanuc_arcmate120id_support/meshes/arcmate120id12l/collision/base_link.stl"/>
+          <mesh filename="package://fanuc_m20id_support/meshes/m20id/collision/base_link.stl"/>
         </geometry>
       </collision>
@@ -25,5 +23,5 @@
         <origin xyz="0 0 0" rpy="0 0 0"/>
         <geometry>
-          <mesh filename="package://fanuc_arcmate120id_support/meshes/arcmate120id12l/visual/link_1.stl"/>
+          <mesh filename="package://fanuc_m20id_support/meshes/m20id/visual/link_1.stl"/>
         </geometry>
         <xacro:material_fanuc_yellow/>
@@ -32,5 +30,5 @@
         <origin xyz="0 0 0" rpy="0 0 0"/>
         <geometry>
-          <mesh filename="package://fanuc_arcmate120id_support/meshes/arcmate120id12l/collision/link_1.stl"/>
+          <mesh filename="package://fanuc_m20id_support/meshes/m20id/collision/link_1.stl"/>
         </geometry>
       </collision>
@@ -40,5 +38,5 @@
         <origin xyz="0 0 0" rpy="0 0 0"/>
         <geometry>
-          <mesh filename="package://fanuc_arcmate120id_support/meshes/arcmate120id12l/visual/link_2.stl"/>
+          <mesh filename="package://fanuc_m20id_support/meshes/m20id/visual/link_2.stl"/>
         </geometry>
         <xacro:material_fanuc_black/>
@@ -47,5 +45,5 @@
         <origin xyz="0 0 0" rpy="0 0 0"/>
         <geometry>
-          <mesh filename="package://fanuc_arcmate120id_support/meshes/arcmate120id12l/collision/link_2.stl"/>
+          <mesh filename="package://fanuc_m20id_support/meshes/m20id/collision/link_2.stl"/>
         </geometry>
       </collision>
@@ -55,5 +53,5 @@
         <origin xyz="0 0 0" rpy="0 0 0"/>
         <geometry>
-          <mesh filename="package://fanuc_arcmate120id_support/meshes/arcmate120id12l/visual/link_3.stl"/>
+          <mesh filename="package://fanuc_m20id_support/meshes/m20id/visual/link_3.stl"/>
         </geometry>
         <xacro:material_fanuc_yellow/>
@@ -62,5 +60,5 @@
         <origin xyz="0 0 0" rpy="0 0 0"/>
         <geometry>
-          <mesh filename="package://fanuc_arcmate120id_support/meshes/arcmate120id12l/collision/link_3.stl"/>
+          <mesh filename="package://fanuc_m20id_support/meshes/m20id/collision/link_3.stl"/>
         </geometry>
       </collision>
@@ -70,5 +68,5 @@
         <origin xyz="0 0 0" rpy="0 0 0"/>
         <geometry>
-          <mesh filename="package://fanuc_arcmate120id_support/meshes/arcmate120id12l/visual/link_4.stl"/>
+          <mesh filename="package://fanuc_m20id_support/meshes/m20id/visual/link_4.stl"/>
         </geometry>
         <xacro:material_fanuc_black/>
@@ -77,5 +75,5 @@
         <origin xyz="0 0 0" rpy="0 0 0"/>
         <geometry>
-          <mesh filename="package://fanuc_arcmate120id_support/meshes/arcmate120id12l/collision/link_4.stl"/>
+          <mesh filename="package://fanuc_m20id_support/meshes/m20id/collision/link_4.stl"/>
         </geometry>
       </collision>
@@ -85,5 +83,5 @@
         <origin xyz="0 0 0" rpy="0 0 0"/>
         <geometry>
-          <mesh filename="package://fanuc_arcmate120id_support/meshes/arcmate120id12l/visual/link_5.stl"/>
+          <mesh filename="package://fanuc_m20id_support/meshes/m20id/visual/link_5.stl"/>
         </geometry>
         <xacro:material_fanuc_yellow/>
@@ -92,5 +90,5 @@
         <origin xyz="0 0 0" rpy="0 0 0"/>
         <geometry>
-          <mesh filename="package://fanuc_arcmate120id_support/meshes/arcmate120id12l/collision/link_5.stl"/>
+          <mesh filename="package://fanuc_m20id_support/meshes/m20id/collision/link_5.stl"/>
         </geometry>
       </collision>
@@ -100,5 +98,5 @@
         <origin xyz="0 0 0" rpy="0 0 0"/>
         <geometry>
-          <mesh filename="package://fanuc_arcmate120id_support/meshes/arcmate120id12l/visual/link_6.stl"/>
+          <mesh filename="package://fanuc_m20id_support/meshes/m20id/visual/link_6.stl"/>
         </geometry>
         <xacro:material_fanuc_black/>
@@ -107,5 +105,5 @@
         <origin xyz="0 0 0" rpy="0 0 0"/>
         <geometry>
-          <mesh filename="package://fanuc_arcmate120id_support/meshes/arcmate120id12l/collision/link_6.stl"/>
+          <mesh filename="package://fanuc_m20id_support/meshes/m20id/collision/link_6.stl"/>
         </geometry>
       </collision>
@@ -145,5 +143,5 @@
       <child link="${prefix}link_5"/>
       <axis xyz="0 0 1"/>
-      <limit effort="0" lower="${radians(-140)}" upper="${radians(140)}" velocity="${radians(450)}"/>
+      <limit effort="0" lower="${radians(-140)}" upper="${radians(140)}" velocity="${radians(420)}"/>
     </joint>
     <joint name="${prefix}joint_6" type="revolute">

Commit message: uncommented flanges and tool0 joints

File: fanuc_m20id_support/urdf/m20id12l_macro.xacro (robot description, xacro)
@@ -162,14 +162,11 @@
     </joint>
     <!-- ROS-Industrial 'flange' frame: attachment point for EEF models -->
-    <!--
     <link name="${prefix}flange"/>
     <joint name="${prefix}joint_6-flange" type="fixed">
-      <origin xyz="0 0 0" rpy="0 0 0"/>
+      <origin xyz="0 0 0.0203" rpy="0 0 0"/>
       <parent link="${prefix}link_6"/>
       <child link="${prefix}flange"/>
     </joint>
-    -->
     <!-- ROS-Industrial 'tool0' frame: all-zeros tool frame -->
-    <!--
     <link name="${prefix}tool0"/>
     <joint name="${prefix}link_6-tool0" type="fixed">
@@ -178,5 +175,4 @@
       <child link="${prefix}tool0"/>
     </joint>
-    -->
   </xacro:macro>
 </robot>

File: fanuc_m20id_support/urdf/m20id_macro.xacro (robot description, xacro)
@@ -160,14 +160,11 @@
     </joint>
     <!-- ROS-Industrial 'flange' frame: attachment point for EEF models -->
-    <!--
     <link name="${prefix}flange"/>
     <joint name="${prefix}joint_6-flange" type="fixed">
-      <origin xyz="0 0 0" rpy="0 0 0"/>
+      <origin xyz="0 0 0.0203" rpy="0 0 0"/>
       <parent link="${prefix}link_6"/>
       <child link="${prefix}flange"/>
     </joint>
-    -->
     <!-- ROS-Industrial 'tool0' frame: all-zeros tool frame -->
-    <!--
     <link name="${prefix}tool0"/>
     <joint name="${prefix}link_6-tool0" type="fixed">
@@ -176,5 +173,4 @@
       <child link="${prefix}tool0"/>
     </joint>
-    -->
   </xacro:macro>
 </robot>

Commit message: fixed joint axes

File: fanuc_m20id_support/urdf/m20id12l_macro.xacro (robot description, xacro)
@@ -123,5 +123,5 @@
       <parent link="${prefix}link_1"/>
       <child link="${prefix}link_2"/>
-      <axis xyz="0 0 1"/>
+      <axis xyz="0 0 -1"/>
       <limit effort="0" lower="${radians(-100)}" upper="${radians(160)}" velocity="${radians(210)}"/>
     </joint>
@@ -130,5 +130,5 @@
       <parent link="${prefix}link_2"/>
       <child link="${prefix}link_3"/>
-      <axis xyz="0 0 1"/>
+      <axis xyz="0 0 -1"/>
       <limit effort="0" lower="${radians(-190)}" upper="${radians(268.4)}" velocity="${radians(265)}"/>
     </joint>
@@ -137,5 +137,5 @@
       <parent link="${prefix}link_3"/>
       <child link="${prefix}link_4"/>
-      <axis xyz="0 0 1"/>
+      <axis xyz="0 0 -1"/>
       <limit effort="0" lower="${radians(-200)}" upper="${radians(200)}" velocity="${radians(420)}"/>
     </joint>
@@ -144,5 +144,5 @@
       <parent link="${prefix}link_4"/>
       <child link="${prefix}link_5"/>
-      <axis xyz="0 0 1"/>
+      <axis xyz="0 0 -1"/>
       <limit effort="0" lower="${radians(-140)}" upper="${radians(140)}" velocity="${radians(450)}"/>
     </joint>
@@ -151,5 +151,5 @@
       <parent link="${prefix}link_5"/>
       <child link="${prefix}link_6"/>
-      <axis xyz="0 0 1"/>
+      <axis xyz="0 0 -1"/>
       <limit effort="0" lower="${radians(-270)}" upper="${radians(270)}" velocity="${radians(720)}"/>
     </joint>

File: fanuc_m20id_support/urdf/m20id_macro.xacro (robot description, xacro)
@@ -121,5 +121,5 @@
       <parent link="${prefix}link_1"/>
       <child link="${prefix}link_2"/>
-      <axis xyz="0 0 1"/>
+      <axis xyz="0 0 -1"/>
       <limit effort="0" lower="${radians(-100)}" upper="${radians(160)}" velocity="${radians(210)}"/>
     </joint>
@@ -128,5 +128,5 @@
       <parent link="${prefix}link_2"/>
       <child link="${prefix}link_3"/>
-      <axis xyz="0 0 1"/>
+      <axis xyz="0 0 -1"/>
       <limit effort="0" lower="${radians(-190)}" upper="${radians(268.4)}" velocity="${radians(265)}"/>
     </joint>
@@ -135,5 +135,5 @@
       <parent link="${prefix}link_3"/>
       <child link="${prefix}link_4"/>
-      <axis xyz="0 0 1"/>
+      <axis xyz="0 0 -1"/>
       <limit effort="0" lower="${radians(-200)}" upper="${radians(200)}" velocity="${radians(420)}"/>
     </joint>
@@ -142,5 +142,5 @@
       <parent link="${prefix}link_4"/>
       <child link="${prefix}link_5"/>
-      <axis xyz="0 0 1"/>
+      <axis xyz="0 0 -1"/>
       <limit effort="0" lower="${radians(-140)}" upper="${radians(140)}" velocity="${radians(420)}"/>
     </joint>
@@ -149,5 +149,5 @@
       <parent link="${prefix}link_5"/>
       <child link="${prefix}link_6"/>
-      <axis xyz="0 0 1"/>
+      <axis xyz="0 0 -1"/>
       <limit effort="0" lower="${radians(-270)}" upper="${radians(270)}" velocity="${radians(720)}"/>
     </joint>
